Commit message: Fix Gazebo startup delay, physics crash, and unreachable hole position
Three bugs:
1. GAZEBO_MODEL_DATABASE_URI not suppressed: Gazebo attempted to fetch the
   online Fuel model catalogue at every startup, causing a multi-minute
   "Preparing your world..." hang even when models are cached locally.
   Fix: SetEnvironmentVariable('GAZEBO_MODEL_DATABASE_URI', '') in launch.

2. Degenerate ground_plane collision in URDF: the xacro:if sim_gazebo block
   added a fixed link with <box size="5 5 0"/> (zero Z) as a collision shape.
   ODE's solver produces large corrective forces for zero-volume bodies,
   physically pushing the robot entity into the ground on spawn.
   Fix: remove the URDF ground_plane link entirely; the world file already
   provides model://ground_plane.

3. Hole placed at x=-0.80, z=0.45 – behind the robot and at distance ≈0.92 m,
   exceeding the UR5e's 0.85 m reach.  Insertion pipeline would always fail.
   Fix: move to x=0.55, z=0.40 (in front of the robot; insertion TCP travels
   to x=0.60 at distance 0.72 m).  Also reversed insertion direction to +X
   (approach from −X side) and updated success criterion accordingly.

Co-Authored-By: Claude Sonnet 4.6 <noreply@anthropic.com>

File: src/peg_in_hole_description/urdf/ur5e_robotiq85.urdf.xacro (robot description, xacro)
@@ -24,22 +24,4 @@
   <!-- World link -->
   <link name="world"/>
-  <!-- Ground plane (Gazebo only) -->
-  <xacro:if value="$(arg sim_gazebo)">
-    <link name="ground_plane">
-      <visual>
-        <origin rpy="0 0 0" xyz="0 0 0"/>
-        <geometry><box size="5 5 0"/></geometry>
-      </visual>
-      <collision>
-        <origin rpy="0 0 0" xyz="0 0 0"/>
-        <geometry><box size="5 5 0"/></geometry>
-      </collision>
-    </link>
-    <joint name="ground_plane_joint" type="fixed">
-      <origin xyz="0 0 -0.01" rpy="0 0 0"/>
-      <parent link="world"/>
-      <child link="ground_plane"/>
-    </joint>
-  </xacro:if>
   <!-- UR arm -->
   <xacro:ur_robot
